File: KiCAD/lf_wobbulator.sch (KiCad schematic (older format))
At the start: 27 parts, among them J1 H_PGA, J2 DDS_OUT, J3 H_SPI, J4 H_VOUT, J5 ADC_IN, J6 H_ADC_IO, J7 H_ADC_I2C, U1 Raspi_Pico, U2 MAX4167

Commit message: all in modules, e-paper added
Parts:
- removed R?: 10k, symbol weigu:R
- added C?: 100µ, symbol weigu:C+
- added J?: DDS_OUT_BI, symbol weigu:SIL1x2L
- added R?: 10k, symbol weigu:R
- added SW?: Kill_DC, symbol weigu:Switch_Closer
- added U?: AD8052, symbol weigu:AD8052
- U2: value MAX4167 -> AD8052; symbol weigu:MAX4167 -> weigu:AD8052
Connections:
- net GND: now also J1.1 (11), J2.2 (12), J?.2 (12), U?.5 (+)
- net at J1.2 (12), J2.1 (11): now also C?.1, SW?.2
- net at D1.2 (A), U2.1: now also U2.2 (-); no longer R?.2
- net at R?.1: now also C?.2, SW?.1; no longer U2.2 (-)
- net at U2.3 (+): now also J5.1 (11); no longer R?.1
- net at C?.1, R?.1, U?.5 (VOUT): no longer U2.4 (V-)
- net at R?.2: now also R?.2, R?.1, U?.6 (-); no longer J5.1 (11)
- net at RV?.~: now also R?.2
- new net: J?.1 (11), R?.1, U?.7
Other:
- moved on the sheet: C1, C2, C3, C4, C?, D1, D?, J1, J2, J3, J4, J5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
